File: hardware/dc-protect-tilted-x804/dc-protect.kicad_sch (KiCad schematic)
At the start: 6 parts, among them P1 CON-SENSOR2-BLANK, U1 DC-Protect

Commit message: Hardware: dc-protect-tilted-x804 V1.4 Added 2 DNP-C footprints, Pin 7 disconnect, added fiducials
Parts:
- added C5: DNP, kicad-libraries:C0805E, symbol tinkerforge:C
- added C6: DNP, kicad-libraries:C0402E, symbol tinkerforge:C
Connections:
- net GND: now also C5.1, C6.1
- net at P1.6, U1.6 (VCC): now also C5.2, C6.2
- net at U1.7 (PWM-OUT): no longer P1.7
- no-connect marks 0 -> 2
Changed lines of the file:
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@@
   (junction (at 146.05 93.98) (diameter 0) (color 0 0 0 0)
   )
+  (junction (at 132.08 92.71) (diameter 0) (color 0 0 0 0)
+  )
+  (junction (at 121.92 92.71) (diameter 0) (color 0 0 0 0)
+  )
   (junction (at 179.07 93.98) (diameter 0) (color 0 0 0 0)
   )
+  (junction (at 132.08 102.87) (diameter 0) (color 0 0 0 0)
+  )
+  (junction (at 121.92 102.87) (diameter 0) (color 0 0 0 0)
+  )
   (junction (at 190.5 86.36) (diameter 0) (color 0 0 0 0)
   )
@@
   (junction (at 198.12 93.98) (diameter 0) (color 0 0 0 0)
   )
+  (no_connect (at 213.36 101.6))
+  (no_connect (at 114.3 97.79))
   (wire (pts (xy 132.08 78.74) (xy 166.37 78.74))
     (stroke (width 0) (type default) (color 0 0 0 0))
@@
     (stroke (width 0) (type default) (color 0 0 0 0))
   )
-  (wire (pts (xy 138.43 97.79) (xy 213.36 97.79))
-    (stroke (width 0) (type default) (color 0 0 0 0))
-  )
   (wire (pts (xy 146.05 92.71) (xy 146.05 93.98))
     (stroke (width 0) (type default) (color 0 0 0 0))
   )
-  (wire (pts (xy 132.08 97.79) (xy 132.08 101.6))
-    (stroke (width 0) (type default) (color 0 0 0 0))
-  )
-  (wire (pts (xy 138.43 97.79) (xy 138.43 95.25))
+  (wire (pts (xy 121.92 92.71) (xy 132.08 92.71))
+    (stroke (width 0) (type default) (color 0 0 0 0))
+  )
+  (wire (pts (xy 132.08 92.71) (xy 146.05 92.71))
     (stroke (width 0) (type default) (color 0 0 0 0))
   )
@@
     (stroke (width 0) (type default) (color 0 0 0 0))
   )
+  (wire (pts (xy 121.92 102.87) (xy 132.08 102.87))
+    (stroke (width 0) (type default) (color 0 0 0 0))
+  )
   (wire (pts (xy 146.05 93.98) (xy 166.37 93.98))
     (stroke (width 0) (type default) (color 0 0 0 0))
@@
     (stroke (width 0) (type default) (color 0 0 0 0))
   )
-  (wire (pts (xy 114.3 97.79) (xy 132.08 97.79))
-    (stroke (width 0) (type default) (color 0 0 0 0))
-  )
-  (wire (pts (xy 132.08 101.6) (xy 213.36 101.6))
+  (wire (pts (xy 132.08 102.87) (xy 208.28 102.87))
     (stroke (width 0) (type default) (color 0 0 0 0))
   )
@@
     (stroke (width 0) (type default) (color 0 0 0 0))
   )
+  (wire (pts (xy 116.84 102.87) (xy 121.92 102.87))
+    (stroke (width 0) (type default) (color 0 0 0 0))
+  )
   (wire (pts (xy 198.12 100.33) (xy 198.12 93.98))
     (stroke (width 0) (type default) (color 0 0 0 0))
@@
     (stroke (width 0) (type default) (color 0 0 0 0))
   )
-  (wire (pts (xy 114.3 92.71) (xy 146.05 92.71))
-    (stroke (width 0) (type default) (color 0 0 0 0))
-  )
-  (wire (pts (xy 138.43 95.25) (xy 114.3 95.25))
+  (wire (pts (xy 114.3 92.71) (xy 121.92 92.71))
     (stroke (width 0) (type default) (color 0 0 0 0))
   )
@@
     (stroke (width 0) (type default) (color 0 0 0 0))
   )
+  (wire (pts (xy 116.84 102.87) (xy 116.84 95.25))
+    (stroke (width 0) (type default) (color 0 0 0 0))
+  )
   (wire (pts (xy 184.15 93.98) (xy 198.12 93.98))
     (stroke (width 0) (type default) (color 0 0 0 0))
   )
+  (wire (pts (xy 208.28 97.79) (xy 208.28 102.87))
+    (stroke (width 0) (type default) (color 0 0 0 0))
+  )
   (wire (pts (xy 114.3 90.17) (xy 203.2 90.17))
     (stroke (width 0) (type default) (color 0 0 0 0))
@@
     (stroke (width 0) (type default) (color 0 0 0 0))
   )
+  (wire (pts (xy 213.36 97.79) (xy 208.28 97.79))
+    (stroke (width 0) (type default) (color 0 0 0 0))
+  )
   (wire (pts (xy 179.07 82.55) (xy 213.36 82.55))
     (stroke (width 0) (type default) (color 0 0 0 0))
@@
   )
   (wire (pts (xy 198.12 93.98) (xy 213.36 93.98))
+    (stroke (width 0) (type default) (color 0 0 0 0))
+  )
+  (wire (pts (xy 114.3 95.25) (xy 116.84 95.25))
     (stroke (width 0) (type default) (color 0 0 0 0))
   )
@@
     (pin "2")
   )
+  (symbol (lib_id "tinkerforge:C") (at 121.92 97.79 0) (unit 1)
+    (in_bom yes) (on_board yes) (fields_autoplaced)
+    (property "Reference" "C5" (id 0) (at 125.222 96.9553 0)
+      (effects (font (size 1.27 1.27)) (justify left))
+    )
+    (property "Value" "DNP" (id 1) (at 125.222 99.4922 0)
+      (effects (font (size 1.27 1.27)) (justify left))
+    )
+    (property "Footprint" "kicad-libraries:C0805E" (id 2) (at 121.92 97.79 0)
+      (effects (font (size 1.524 1.524)) hide)
+    )
+    (property "Datasheet" "" (id 3) (at 121.92 97.79 0)
+      (effects (font (size 1.524 1.524)))
+    )
+    (pin "1")
+    (pin "2")
+  )
   (symbol (lib_id "tinkerforge:C") (at 203.2 95.25 0) (unit 1)
     (in_bom yes) (on_board yes) (fields_autoplaced)
@@
     )
     (property "Datasheet" "" (id 3) (at 190.5 91.44 0)
+      (effects (font (size 1.524 1.524)))
+    )
+    (pin "1")
+    (pin "2")
+  )
+  (symbol (lib_id "tinkerforge:C") (at 132.08 97.79 0) (unit 1)
+    (in_bom yes) (on_board yes) (fields_autoplaced)
+    (property "Reference" "C6" (id 0) (at 135.382 96.9553 0)
+      (effects (font (size 1.27 1.27)) (justify left))
+    )
+    (property "Value" "DNP" (id 1) (at 135.382 99.4922 0)
+      (effects (font (size 1.27 1.27)) (justify left))
+    )
+    (property "Footprint" "kicad-libraries:C0402E" (id 2) (at 132.08 97.79 0)
+      (effects (font (size 1.524 1.524)) hide)
+    )
+    (property "Datasheet" "" (id 3) (at 132.08 97.79 0)
       (effects (font (size 1.524 1.524)))
     )
@@
       (reference "C4") (unit 1) (value "100nF") (footprint "kicad-libraries:C0402E")
     )
+    (path "/124632df-682f-4e38-bc1f-099b1dea3d5a"
+      (reference "C5") (unit 1) (value "DNP") (footprint "kicad-libraries:C0805E")
+    )
+    (path "/feefa11c-ae77-499b-b8b6-277a18b389b2"
+      (reference "C6") (unit 1) (value "DNP") (footprint "kicad-libraries:C0402E")
+    )
     (path "/00000000-0000-0000-0000-000060362595"

Commit message: fix dc protect outline, move to mm (54x60)
Other:
- note added: "Copyright Tinkerforge GmbH 2023. This documentation describes Open Hardware and is licensed under the CERN OHL v. 1.1. You may redistribute and modify this documentation under the terms of the CERN OHL v.1.1. (http://ohwr.org/cernohl). This documentation is distributed WITHOUT ANY EXPRESS OR IMPLIED WARRANTY, INCLUDING OF MERCHANTABILITY, SATISFACTORY QUALITY AND FITNESS FOR A PARTICULAR PURPOSE.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"
- note removed: "Copyright Tinkerforge GmbH 2021. This documentation describes Open Hardware and is licensed under the CERN OHL v. 1.1. You may redistribute and modify this documentation under the terms of the CERN OHL v.1.1. (http://ohwr.org/cernohl). This documentation is distributed WITHOUT ANY EXPRESS OR IMPLIED WARRANTY, INCLUDING OF MERCHANTABILITY, SATISFACTORY QUALITY AND FITNESS FOR A PARTICULAR PURPOSE.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"
- title: DC Protect -> DC Protect Tilted X804
Changed lines of the file:
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@@
   (paper "A4")
   (title_block
-    (title "DC Protect")
-    (date "2022-12-07")
-    (rev "1.3")
+    (title "DC Protect Tilted X804")
+    (date "2023-02-03")
+    (rev "1.4")
     (company "Tinkerforge GmbH")
     (comment 1 "Licensed under CERN OHL v.1.1")
-    (comment 2 "Copyright (©) 2020, T.Schneidermann <tim@tinkerforge.com>")
+    (comment 2 "Copyright (©) 2023, T.Schneidermann <tim@tinkerforge.com>")
   )
   (junction (at 184.15 93.98) (diameter 0) (color 0 0 0 0)
@@
     (stroke (width 0) (type default) (color 0 0 0 0))
   )
-  (text "Copyright Tinkerforge GmbH 2021.\nThis documentation describes Open Hardware and is licensed under the\nCERN OHL v. 1.1.\nYou may redistribute and modify this documentation under the terms of the\nCERN OHL v.1.1. (http://ohwr.org/cernohl). This documentation is distributed\nWITHOUT ANY EXPRESS OR IMPLIED WARRANTY, INCLUDING OF\nMERCHANTABILITY, SATISFACTORY QUALITY AND FITNESS FOR A\nPARTICULAR PURPOSE. Please see the CERN OHL v.1.1 for applicable\nconditions\n"
+  (text "Copyright Tinkerforge GmbH 2023.\nThis documentation describes Open Hardware and is licensed under the\nCERN OHL v. 1.1.\nYou may redistribute and modify this documentation under the terms of the\nCERN OHL v.1.1. (http://ohwr.org/cernohl). This documentation is distributed\nWITHOUT ANY EXPRESS OR IMPLIED WARRANTY, INCLUDING OF\nMERCHANTABILITY, SATISFACTORY QUALITY AND FITNESS FOR A\nPARTICULAR PURPOSE. Please see the CERN OHL v.1.1 for applicable\nconditions\n"
     (at 12.7 196.85 0)
     (effects (font (size 1.016 1.016)) (justify left bottom))
